Commit message: init foxy

File: velodyne_description/urdf/HDL-32E.urdf.xacro (robot description, xacro)
@@ -2,5 +2,5 @@
 <robot xmlns:xacro="http://www.ros.org/wiki/xacro" name="HDL-32E">
   <xacro:property name="M_PI" value="3.1415926535897931" />
-  <xacro:macro name="HDL-32E" params="*origin parent:=base_link name:=velodyne topic:=/velodyne_points hz:=10 lasers:=32 samples:=2187 collision_range:=0.3 min_range:=0.9 max_range:=130.0 noise:=0.008 min_angle:=-${M_PI} max_angle:=${M_PI} gpu:=false">
+  <xacro:macro name="HDL-32E" params="*origin parent:=base_link name:=velodyne tf_prefix:='' topic:=/velodyne_points organize_cloud:=false hz:=10 lasers:=32 samples:=2187 collision_range:=0.3 min_range:=0.9 max_range:=130.0 noise:=0.008 min_angle:=-${M_PI} max_angle:=${M_PI} gpu:=false">
     <joint name="${name}_base_mount_joint" type="fixed">
       <xacro:insert_block name="origin" />
@@ -45,4 +45,9 @@
         </geometry>
       </visual>
+      <collision>
+        <geometry>
+          <sphere radius="0"/>
+        </geometry>
+      </collision>
     </link>
     <!-- Gazebo requires the velodyne_gazebo_plugins package -->
@@ -79,10 +84,15 @@
             </noise>
           </ray>
-          <plugin name="gazebo_ros_laser_controller" filename="libgazebo_ros_velodyne_gpu_laser.so">
-            <topicName>${topic}</topicName>
-            <frameName>${name}</frameName>
+          <plugin name="gazebo_ros_laser_controller" filename="libgazebo_ros_velodyne_laser.so">
+            <ros>
+              <namespace>/${name}</namespace>
+              <remapping>~/out:=${topic}</remapping>
+            </ros>
+            <tf_prefix>${tf_prefix}</tf_prefix>
+            <frame_name>${name}</frame_name>
+            <organize_cloud>${organize_cloud}</organize_cloud>
             <min_range>${min_range}</min_range>
             <max_range>${max_range}</max_range>
-            <gaussianNoise>${noise}</gaussianNoise>
+            <gaussian_noise>${noise}</gaussian_noise>
           </plugin>
         </sensor>
@@ -120,9 +130,14 @@
           </ray>
           <plugin name="gazebo_ros_laser_controller" filename="libgazebo_ros_velodyne_laser.so">
-            <topicName>${topic}</topicName>
-            <frameName>${name}</frameName>
+            <ros>
+              <namespace>/${name}</namespace>
+              <remapping>~/out:=${topic}</remapping>
+            </ros>
+            <tf_prefix>${tf_prefix}</tf_prefix>
+            <frame_name>${name}</frame_name>
+            <organize_cloud>${organize_cloud}</organize_cloud>
             <min_range>${min_range}</min_range>
             <max_range>${max_range}</max_range>
-            <gaussianNoise>${noise}</gaussianNoise>
+            <gaussian_noise>${noise}</gaussian_noise>
           </plugin>
         </sensor>

File: velodyne_description/urdf/VLP-16.urdf.xacro (robot description, xacro)
@@ -2,5 +2,5 @@
 <robot xmlns:xacro="http://www.ros.org/wiki/xacro" name="VLP-16">
   <xacro:property name="M_PI" value="3.1415926535897931" />
-  <xacro:macro name="VLP-16" params="*origin parent:=base_link name:=velodyne topic:=/velodyne_points hz:=10 lasers:=16 samples:=1875 collision_range:=0.3 min_range:=0.9 max_range:=130.0 noise:=0.008 min_angle:=-${M_PI} max_angle:=${M_PI} gpu:=false">
+  <xacro:macro name="VLP-16" params="*origin parent:=base_link name:=velodyne tf_prefix:='' topic:=/velodyne_points organize_cloud:=false hz:=10 lasers:=16 samples:=1875 collision_range:=0.3 min_range:=0.9 max_range:=130.0 noise:=0.008 min_angle:=-${M_PI} max_angle:=${M_PI} gpu:=false">
     <joint name="${name}_base_mount_joint" type="fixed">
       <xacro:insert_block name="origin" />
@@ -50,4 +50,9 @@
         </geometry>
       </visual>
+      <collision>
+        <geometry>
+          <sphere radius="0"/>
+        </geometry>
+      </collision>
     </link>
     <!-- Gazebo requires the velodyne_gazebo_plugins package -->
@@ -84,10 +89,15 @@
             </noise>
           </ray>
-          <plugin name="gazebo_ros_laser_controller" filename="libgazebo_ros_velodyne_gpu_laser.so">
-            <topicName>${topic}</topicName>
-            <frameName>${name}</frameName>
+          <plugin name="gazebo_ros_laser_controller" filename="libgazebo_ros_velodyne_laser.so">
+            <ros>
+              <namespace>/${name}</namespace>
+              <remapping>~/out:=${topic}</remapping>
+            </ros>
+            <tf_prefix>${tf_prefix}</tf_prefix>
+            <frame_name>${name}</frame_name>
+            <organize_cloud>${organize_cloud}</organize_cloud>
             <min_range>${min_range}</min_range>
             <max_range>${max_range}</max_range>
-            <gaussianNoise>${noise}</gaussianNoise>
+            <gaussian_noise>${noise}</gaussian_noise>
           </plugin>
         </sensor>
@@ -125,9 +135,14 @@
           </ray>
           <plugin name="gazebo_ros_laser_controller" filename="libgazebo_ros_velodyne_laser.so">
-            <topicName>${topic}</topicName>
-            <frameName>${name}</frameName>
+            <ros>
+              <namespace>/${name}</namespace>
+              <remapping>~/out:=${topic}</remapping>
+            </ros>
+            <tf_prefix>${tf_prefix}</tf_prefix>
+            <frame_name>${name}</frame_name>
+            <organize_cloud>${organize_cloud}</organize_cloud>
             <min_range>${min_range}</min_range>
             <max_range>${max_range}</max_range>
-            <gaussianNoise>${noise}</gaussianNoise>
+            <gaussian_noise>${noise}</gaussian_noise>
           </plugin>
         </sensor>
